File: electronics/register_board/register_board.kicad_pcb (KiCad board)
At the start: 4 copper layers, 160 x 100 mm, 151 parts, among them CN1 4-2271013-0, U1 74HC00, U10 SN74HC574PWR, U11 SN74HC574PWR, U12 SN74HC574PWR, U13 SN74HC574PWR, U14 SN74HC574PWR, U15 SN74HC574PWR, U16 SN74HC574PWR, U17 SN74HC574PWR, U18 SN74HC574PWR, U19 SN74HC574PWR, U2 74HC157, U20 SN74HC574PWR, U21 SN74HC574PWR, U22 SN74HC574PWR, U23 SN74HC574PWR, U24 SN74HC574PWR, U25 SN74HC574PWR, U26 SN74HC574PWR, U27 SN74HC574PWR, U28 SN74HC574PWR, U29 SN74HC574PWR, U3 74HC138, U30 SN74HC574PWR, U31 SN74HC574PWR, U32 SN74HC574PWR, U33 SN74HC574PWR, U34 SN74HC574PWR, U35 SN74HC574PWR, U36 SN74HC574PWR, U37 SN74HC574PWR, U38 SN74HC574PWR, U39 SN74HC574PWR, U4 74HC138, U40 SN74HC574PWR, U41 SN74HC574PWR, U42 SN74HC574PWR, U43 SN74HC574PWR, U44 SN74HC574PWR, U45 SN74HC574PWR, U46 SN74HC574PWR, U47 SN74HC574PWR, U48 SN74HC574PWR, U49 SN74HC574PWR, U5 74HC138, U50 SN74HC574PWR, U51 SN74HC574PWR, U52 SN74HC574PWR, U53 SN74HC574PWR, U54 SN74HC574PWR, U55 SN74HC574PWR, U56 SN74HC574PWR, U57 SN74HC574PWR, U58 SN74HC574PWR, U59 SN74HC574PWR, U6 74HC138, U60 SN74HC574PWR, U61 SN74HC574PWR, U62 SN74HC574PWR, U63 SN74HC574PWR, U64 SN74HC574PWR, U65 SN74HC574PWR, U66 SN74HC574PWR, U67 SN74HC574PWR, U68 SN74HC574PWR, U69 SN74HC574PWR, U7 74HC138, U70 SN74HC574PWR, U71 SN74HC574PWR, U72 SN74HC574PWR, U73 SN74HC574PWR, U74 SN74HC574PWR, U8 74HC138, U9 SN74HC574PWR

Commit message: Updated WIP register board PCB
Parts:
- added C75: 100nF, Capacitor_SMD:C_0603_1608Metric, F.Cu at (277.7, 112.6)
- added U75: SN74HC574PWR, easyeda2kicad:TSSOP-20_L6.5-W4.4-P0.65-LS6.4-BL, F.Cu at (280.1, 107.1)
Connections:
- net /D_SEL0 renamed /D_SEL_LATCHED0
- net /D_SEL1 renamed /D_SEL_LATCHED1
- net /D_SEL2 renamed /D_SEL_LATCHED2
- net /D_SEL3 renamed /D_SEL_LATCHED3
- net /LOAD renamed /LOAD_LATCHED
- net /~{RESET} renamed /RESET
